Commit message: bimur manipulation

File: bimur_description/urdf/bimur_right_arm.urdf (robot description, URDF)
Before this commit: robot ur5, 22 links, 21 joints
Links:
- link frame: geometry collision mesh filename=package://bimur_description/meshes/UR5Frame.STL; visual mesh filename=package://bimur_description/meshes/UR5Frame.STL

File: bimur_description/urdf/bimur_right_arm.xacro (robot description, xacro)
@@ -26,5 +26,5 @@
       <origin rpy="0.0 0 0" xyz="0 0 0"/>
       <geometry>
-        <mesh filename="package://bimur_description/meshes/objects/UR5Frame.STL"/>
+        <mesh filename="package://bimur_description/meshes/UR5Frame.STL"/>
       </geometry>
     </collision>
@@ -32,5 +32,5 @@
       <origin rpy="0.0 0 0" xyz="0 0 0"/>
       <geometry>
-        <mesh filename="package://bimur_description/meshes/objects/UR5Frame.STL"/>
+        <mesh filename="package://bimur_description/meshes/UR5Frame.STL"/>
       </geometry>
     </visual>
