Commit message: Fixed arm attach angle in URDF

File: bimur_description/urdf/bimur_right_arm.xacro (robot description, xacro)
@@ -73,5 +73,5 @@
     <parent link="frame"/>
     <child link = "base_link"/>
-    <origin xyz="0.265 0.635 1.275" rpy="${0*pi/180} ${225*pi/180}  ${0*pi/180}"/>
+    <origin xyz="0.265 0.635 1.275" rpy="${-45*pi/180} ${180*pi/180}  ${90*pi/180}"/>
   </joint>
 </robot>

Commit message: Updates

File: bimur_description/urdf/bimur_right_arm.xacro (robot description, xacro)
@@ -1,4 +1,5 @@
 <?xml version="1.0"?>
 <robot xmlns:xacro="http://ros.org/wiki/xacro" name="ur5" >
+  <xacro:arg name="transmission_hw_interface" default="hardware_interface/PositionJointInterface"/>
   <!-- common stuff -->
   <xacro:include filename="$(find ur_description)/urdf/common.gazebo.xacro" />
@@ -6,11 +7,13 @@
   <xacro:include filename="$(find ur_description)/urdf/ur5.urdf.xacro" />
   <!-- Right arm -->
-  <xacro:ur5_robot prefix="" joint_limited="false"/>
+  <xacro:ur5_robot prefix="" joint_limited="false"
+    transmission_hw_interface="$(arg transmission_hw_interface)"
+  />
   <!-- robotiq 85 -->
-  <xacro:include filename="$(find robotiq_85_description)/urdf/robotiq_85_gripper.urdf.xacro" />
+<!--   <xacro:include filename="$(find robotiq_85_description)/urdf/robotiq_85_gripper.urdf.xacro" /> -->
   <!-- Right robotiq 85 -->
-  <xacro:robotiq_85_gripper prefix="" parent="ee_link" >
-    <origin xyz="0 0 0" rpy="0 0 0"/>
-  </xacro:robotiq_85_gripper>
+<!--   <xacro:robotiq_85_gripper prefix="" parent="ee_link" >
+    <origin xyz="0.1 0 0" rpy="0 0 0"/>
+  </xacro:robotiq_85_gripper> -->
   <link name="world"/>
   <link name="frame">

Commit message: Updates

File: bimur_description/urdf/bimur_right_arm.xacro (robot description, xacro)
@@ -11,9 +11,9 @@
   />
   <!-- robotiq 85 -->
-<!--   <xacro:include filename="$(find robotiq_85_description)/urdf/robotiq_85_gripper.urdf.xacro" /> -->
+  <xacro:include filename="$(find robotiq_85_description)/urdf/robotiq_85_gripper.urdf.xacro" />
   <!-- Right robotiq 85 -->
-<!--   <xacro:robotiq_85_gripper prefix="" parent="ee_link" >
-    <origin xyz="0.1 0 0" rpy="0 0 0"/>
-  </xacro:robotiq_85_gripper> -->
+  <xacro:robotiq_85_gripper prefix="" parent="ee_link" >
+    <origin xyz="0 0 0" rpy="0 0 0"/>
+  </xacro:robotiq_85_gripper>
   <link name="world"/>
   <link name="frame">

Commit message: Update bimur_right_arm.xacro
Added ramp link and joint to the rest of the URDF

File: bimur_description/urdf/bimur_right_arm.xacro (robot description, xacro)
@@ -59,4 +59,27 @@
     </collision>
   </link>
+    <link name="ramp">
+    <inertial>
+      <origin xyz="0.5 0 0.755" rpy="0 0 0" />
+      <mass value="1"/>
+      <inertia
+        ixx="0.07" ixy="0.0" ixz="0.0"
+        iyy="0.40" iyz="0.0"
+        izz="0.33"/>
+    </inertial>
+    <visual>
+      <geometry>
+        <box size="0.5 0.5 0.05"/>
+      </geometry>
+      <material name="orange">
+        <color rgba="0 0 .8 1"/>
+      </material>
+    </visual>
+    <collision>
+      <geometry>
+        <box size="0.5 0.5 0.05"/>
+      </geometry>
+    </collision>
+  </link>
  <joint name="frame_to_world" type="fixed">
     <parent link="world"/>
@@ -75,3 +98,9 @@
     <origin xyz="0.265 0.635 1.275" rpy="${-45*pi/180} ${180*pi/180}  ${90*pi/180}"/>
   </joint>
+    <!-- ramp -->
+  <joint name="ramp_to_frame" type="fixed">
+    <parent link="frame"/>
+    <child link = "base_link"/>
+    <origin xyz="0.5 0 0.755" rpy="0.0 0.0 0.0"/>
+  </joint>
 </robot>

Commit message: add reference to ramp STL file

File: bimur_description/urdf/bimur_right_arm.xacro (robot description, xacro)
@@ -70,5 +70,5 @@
     <visual>
       <geometry>
-        <box size="0.5 0.5 0.05"/>
+        <mesh filename="package://bimur_description/meshes/ramp.STL"/>
       </geometry>
       <material name="orange">
@@ -78,5 +78,5 @@
     <collision>
       <geometry>
-        <box size="0.5 0.5 0.05"/>
+        <mesh filename="package://bimur_description/meshes/ramp.STL"/>
       </geometry>
     </collision>
