Commit message: Added Astra camera

File: bimur_description/urdf/bimur_right_robot.urdf.xacro (robot description, xacro)
@@ -18,4 +18,7 @@
     <origin xyz="0 0 0" rpy="0 0 0"/>
   </xacro:robotiq_85_gripper>
+  <!-- Astra camera -->
+  <xacro:include filename="$(find bimur_description)/urdf/camera/astra.xacro"/>
+  <xacro:sensor_astra name="astra" parent="camera_mount" cam_px="0.01" cam_pz="${0.052}" meshes="package://bimur_description/meshes/rgbd" />
   <link name="world"/>
   <link name="frame">
@@ -80,3 +83,10 @@
     <origin xyz="0.265 0.635 1.275" rpy="${-45*pi/180} ${180*pi/180}  ${90*pi/180}"/>
   </joint>
+  <!-- astra camera -->
+  <link name="camera_mount"/>
+  <joint name="camera_to_frame" type="fixed">
+    <parent link="frame"/>
+    <child link = "camera_mount"/>
+    <origin xyz="0.5 0.53 1.58" rpy="${0} ${0} ${-PI/2}"/>
+  </joint>
 </robot>

Commit message: Corrected camera orientation in urdf and updated README with how to launch camera driver

File: bimur_description/urdf/bimur_right_robot.urdf.xacro (robot description, xacro)
@@ -88,5 +88,5 @@
     <parent link="frame"/>
     <child link = "camera_mount"/>
-    <origin xyz="0.5 0.53 1.58" rpy="${0} ${0} ${-PI/2}"/>
+    <origin xyz="0.54 0.54 1.54" rpy="${0} ${75*pi/180} ${-pi/2}"/>
   </joint>
 </robot>

Commit message: Added wait for active bag files, updated camera height in urdf, minor code updates

File: bimur_description/urdf/bimur_right_robot.urdf.xacro (robot description, xacro)
@@ -88,5 +88,5 @@
     <parent link="frame"/>
     <child link = "camera_mount"/>
-    <origin xyz="0.54 0.54 1.54" rpy="${0} ${75*pi/180} ${-pi/2}"/>
+    <origin xyz="0.54 0.54 1.45" rpy="${0} ${75*pi/180} ${-pi/2}"/>
   </joint>
 </robot>

Commit message: modified files to run gazebo and moveit

File: bimur_description/urdf/bimur_right_robot.urdf.xacro (robot description, xacro)
@@ -2,7 +2,7 @@
 <robot xmlns:xacro="http://wiki.ros.org/xacro" name="ur5" >
   <!-- common stuff -->
-  <xacro:include filename="$(find ur_description)/urdf/common.gazebo.xacro" />
+  <!-- <xacro:include filename="$(find ur_description)/urdf/common.gazebo.xacro" /> -->
   <!-- ur5 -->
-  <xacro:include filename="$(find ur_description)/urdf/ur5.urdf.xacro" />
+  <xacro:include filename="$(find ur_description)/urdf/ur5.xacro" />
   <!-- Right arm -->
   <xacro:arg name="transmission_hw_interface" default="hardware_interface/PositionJointInterface"/>
@@ -19,6 +19,6 @@
   </xacro:robotiq_85_gripper>
   <!-- Astra camera -->
-  <xacro:include filename="$(find bimur_description)/urdf/camera/astra.xacro"/>
-  <xacro:sensor_astra name="astra" parent="camera_mount" cam_px="0.01" cam_pz="${0.052}" meshes="package://bimur_description/meshes/rgbd" />
+<!--   <xacro:include filename="$(find bimur_description)/urdf/camera/astra.xacro"/>
+  <xacro:sensor_astra name="astra" parent="camera_mount" cam_px="0.01" cam_pz="${0.052}" meshes="package://bimur_description/meshes/rgbd" /> -->
   <link name="world"/>
   <link name="frame">
@@ -84,9 +84,9 @@
   </joint>
   <!-- astra camera -->
-  <link name="camera_mount"/>
+<!--   <link name="camera_mount"/>
   <joint name="camera_to_frame" type="fixed">
     <parent link="frame"/>
     <child link = "camera_mount"/>
     <origin xyz="0.54 0.54 1.45" rpy="${0} ${75*pi/180} ${-pi/2}"/>
-  </joint>
+  </joint> -->
 </robot>
