Commit message: MAJOR UPDATE - new moveit package, new ur driver package

File: robotiq_85_gripper/robotiq_85_description/urdf/robotiq_85_gripper.transmission.xacro (robot description, xacro)
@@ -1,4 +1,4 @@
 <?xml version="1.0"?>
-<robot xmlns:xacro="http://ros.org/wiki/xacro">
+<robot xmlns:xacro="http://wiki.ros.org/xacro">
   <xacro:macro name="robotiq_85_gripper_transmission" params="prefix">
         <transmission name="${prefix}gripper_finger1_trans">

File: robotiq_85_gripper/robotiq_85_description/urdf/robotiq_85_gripper.urdf.xacro (robot description, xacro)
@@ -1,4 +1,4 @@
 <?xml version="1.0"?>
-<robot name="robotiq_85_gripper" xmlns:xacro="http://ros.org/wiki/xacro">
+<robot name="robotiq_85_gripper" xmlns:xacro="http://wiki.ros.org/xacro">
     <xacro:include filename="$(find robotiq_85_description)/urdf/robotiq_85_gripper.transmission.xacro" />
     <xacro:macro name="robotiq_85_gripper" params="prefix parent *origin">
@@ -299,21 +299,4 @@
             <kd>1.0</kd>
         </gazebo>
-	<gazebo>
-	  <plugin name="gazebo_grasp_fix" filename="libgazebo_grasp_fix.so">
-            <arm>
-              <arm_name>gripper_arm</arm_name>
-              <palm_link>${parent}</palm_link>
-              <gripper_link>${prefix}gripper_finger1_finger_tip_link</gripper_link>
-              <gripper_link>${prefix}gripper_finger2_finger_tip_link</gripper_link>
-            </arm>
-	    <forces_angle_tolerance>100</forces_angle_tolerance>
-	    <update_rate>2</update_rate>
-	    <grip_count_threshold>1</grip_count_threshold>
-	    <max_grip_count>2</max_grip_count>
-	    <release_tolerance>0.005</release_tolerance>
-	    <disable_collisions_on_attach>true</disable_collisions_on_attach>
-	    <contact_topic>__default_topic__</contact_topic>
-	  </plugin>
-	</gazebo>
         <xacro:robotiq_85_gripper_transmission prefix="${prefix}" />
     </xacro:macro>

File: robotiq_85_gripper/robotiq_85_description/urdf/robotiq_85_gripper.xacro (robot description, xacro)
@@ -1,4 +1,4 @@
 <?xml version="1.0" ?>
-<robot name="robotiq_85_gripper" xmlns:xacro="http://ros.org/wiki/xacro">
+<robot name="robotiq_85_gripper" xmlns:xacro="http://wiki.ros.org/xacro">
     <xacro:include filename="$(find robotiq_85_description)/urdf/robotiq_85_gripper.urdf.xacro" />
     <gazebo>

File: universal_robot/ur_e_description/urdf/ur10e.urdf.xacro (robot description, xacro)
@@ -25,5 +25,7 @@
     transmission_hw_interface:=hardware_interface/PositionJointInterface
     safety_limits:=false safety_pos_margin:=0.15
-    safety_k_position:=20">
+    safety_k_position:=20
+    kinematics_file">
+    <xacro:property name="__kinematics" value="${kinematics_file['kinematics']}"/>
     <!-- Inertia parameters -->
     <xacro:property name="base_mass" value="4.0" />  <!-- This mass might be incorrect -->
@@ -44,24 +46,13 @@
     <xacro:property name="wrist_2_cog" value="-0.00021 0.00112 0.002269" />
     <xacro:property name="wrist_3_cog" value="0 -0.001156 -0.00149" />
-    <!-- Kinematic model -->
-    <!-- Properties from urcontrol.conf -->
-    <xacro:property name="d1" value="0.181" />
-    <xacro:property name="a2" value="-0.613" />
-    <xacro:property name="a3" value="-0.571" />
-    <xacro:property name="d4" value="0.135" />
-    <xacro:property name="d5" value="0.120" />
-    <xacro:property name="d6" value="0.117" />
     <!-- Arbitrary offsets for shoulder/elbow joints -->
-    <xacro:property name="shoulder_offset" value="0.176" />
-    <xacro:property name="elbow_offset" value="-0.137" />
-    <!-- link lengths used in model -->
-    <xacro:property name="shoulder_height" value="${d1}" />
-    <xacro:property name="upper_arm_length" value="${-a2}" />
-    <xacro:property name="forearm_length" value="${-a3}" />
-    <xacro:property name="wrist_1_length" value="${d4}" />
-    <xacro:property name="wrist_2_length" value="${d5}" />
-    <xacro:property name="wrist_3_length" value="${d6}" />
+    <xacro:property name="shoulder_offset" value="0.1762" />  <!-- measured from model -->
+    <xacro:property name="elbow_offset" value="0.0393" /> <!-- measured from model -->
+    <xacro:property name="upper_arm_inertia_offset" value="0.175" />  <!-- measured from model -->
+    <!-- This is for compatibility reasons, as transformation between base and base_link was always 180 degree in the ur_description -->
+    <xacro:property name="base_correction" value="${pi}" />
     <link name="${prefix}base_link" >
       <visual>
+        <origin xyz="0 0 0" rpy="0 0 ${base_correction}"/>
         <geometry>
           <mesh filename="package://ur_e_description/meshes/ur10e/visual/base.dae"/>
@@ -72,4 +63,5 @@
       </visual>
       <collision>
+        <origin xyz="0 0 0" rpy="0 0 ${base_correction}"/>
         <geometry>
           <mesh filename="package://ur_e_description/meshes/ur10e/collision/base.stl"/>
@@ -83,5 +75,5 @@
       <parent link="${prefix}base_link" />
       <child link = "${prefix}shoulder_link" />
-      <origin xyz="0.0 0.0 ${shoulder_height}" rpy="0.0 0.0 0.0" />
+      <origin xyz="${__kinematics['shoulder']['x']} ${__kinematics['shoulder']['y']} ${__kinematics['shoulder']['z']}" rpy="${__kinematics['shoulder']['roll']} ${__kinematics['shoulder']['pitch']} ${__kinematics['shoulder']['yaw'] + base_correction}" />
       <axis xyz="0 0 1" />
       <xacro:unless value="${joint_limited}">
@@ -101,4 +93,5 @@
     <link name="${prefix}shoulder_link">
       <visual>
+        <origin xyz="0 0 0" rpy="0 0 ${pi}"/>
         <geometry>
           <mesh filename="package://ur_e_description/meshes/ur10e/visual/shoulder.dae"/>
@@ -109,4 +102,5 @@
       </visual>
       <collision>
+        <origin xyz="0 0 0" rpy="0 0 ${pi}"/>
         <geometry>
           <mesh filename="package://ur_e_description/meshes/ur10e/collision/shoulder.stl"/>
@@ -120,6 +114,6 @@
       <parent link="${prefix}shoulder_link" />
       <child link = "${prefix}upper_arm_link" />
-      <origin xyz="0.0 ${shoulder_offset} 0.0" rpy="0.0 ${pi / 2.0} 0.0" />
-      <axis xyz="0 1 0" />
+      <origin xyz="${__kinematics['upper_arm']['x']} ${__kinematics['upper_arm']['y']} ${__kinematics['upper_arm']['z']}" rpy="${__kinematics['upper_arm']['roll']} ${__kinematics['upper_arm']['pitch']} ${__kinematics['upper_arm']['yaw']}" />
+      <axis xyz="0 0 1" />
       <xacro:unless value="${joint_limited}">
         <limit lower="${-2.0 * pi}" upper="${2.0 * pi}" effort="330.0" velocity="3.14"/>
@@ -138,4 +132,5 @@
     <link name="${prefix}upper_arm_link">
       <visual>
+        <origin xyz="0 0 ${shoulder_offset}" rpy="${pi/2} 0 ${-pi/2}"/>
         <geometry>
           <mesh filename="package://ur_e_description/meshes/ur10e/visual/upperarm.dae"/>
@@ -146,10 +141,11 @@
       </visual>
       <collision>
+        <origin xyz="0 0 ${shoulder_offset}" rpy="${pi/2} 0 ${-pi/2}"/>
         <geometry>
           <mesh filename="package://ur_e_description/meshes/ur10e/collision/upperarm.stl"/>
         </geometry>
       </collision>
-      <xacro:cylinder_inertial radius="0.075" length="${-a2}" mass="${upper_arm_mass}">
-        <origin xyz="0.0 0.0 ${-a2/2.0}" rpy="0 0 0" />
+      <xacro:cylinder_inertial radius="0.075" length="${-1*__kinematics['forearm']['x']}" mass="${upper_arm_mass}">
+        <origin xyz="${0.5*__kinematics['forearm']['x']} 0.0 ${upper_arm_inertia_offset}" rpy="0 ${pi/2} 0" />
       </xacro:cylinder_inertial>
     </link>
@@ -157,6 +153,6 @@
       <parent link="${prefix}upper_arm_link" />
       <child link = "${prefix}forearm_link" />
-      <origin xyz="0.0 ${elbow_offset} ${upper_arm_length}" rpy="0.0 0.0 0.0" />
-      <axis xyz="0 1 0" />
+      <origin xyz="${__kinematics['forearm']['x']} ${__kinematics['forearm']['y']} ${__kinematics['forearm']['z']}" rpy="${__kinematics['forearm']['roll']} ${__kinematics['forearm']['pitch']} ${__kinematics['forearm']['yaw']}" />
+      <axis xyz="0 0 1" />
       <xacro:unless value="${joint_limited}">
         <limit lower="${-pi}" upper="${pi}" effort="150.0" velocity="3.14"/>
@@ -175,5 +171,6 @@
     <link name="${prefix}forearm_link">
       <visual>
-         <geometry>
+        <origin xyz="0 0 ${elbow_offset}" rpy="${pi/2} 0 ${-pi/2}"/>
+        <geometry>
           <mesh filename="package://ur_e_description/meshes/ur10e/visual/forearm.dae"/>
         </geometry>
@@ -183,10 +180,11 @@
       </visual>
       <collision>
+        <origin xyz="0 0 ${elbow_offset}" rpy="${pi/2} 0 ${-pi/2}"/>
         <geometry>
           <mesh filename="package://ur_e_description/meshes/ur10e/collision/forearm.stl"/>
         </geometry>
       </collision>
-      <xacro:cylinder_inertial radius="0.075" length="${-a3}" mass="${forearm_mass}">
-        <origin xyz="0.0 0.0 ${-a3/2.0}" rpy="0 0 0" />
+      <xacro:cylinder_inertial radius="0.075" length="${-1*__kinematics['wrist_1']['x']}" mass="${forearm_mass}">
+        <origin xyz="${0.5*__kinematics['forearm']['x']} 0.0 ${elbow_offset}" rpy="0 ${pi/2} 0" />
       </xacro:cylinder_inertial>
     </link>
@@ -194,6 +192,6 @@
       <parent link="${prefix}forearm_link" />
       <child link = "${prefix}wrist_1_link" />
-      <origin xyz="0.0 0.0 ${forearm_length}" rpy="0.0 ${pi / 2.0} 0.0" />
-      <axis xyz="0 1 0" />
+      <origin xyz="${__kinematics['wrist_1']['x']} ${__kinematics['wrist_1']['y']} ${__kinematics['wrist_1']['z']}" rpy="${__kinematics['wrist_1']['roll']} ${__kinematics['wrist_1']['pitch']} ${__kinematics['wrist_1']['yaw']}" />
+      <axis xyz="0 0 1" />
       <xacro:unless value="${joint_limited}">
         <limit lower="${-2.0 * pi}" upper="${2.0 * pi}" effort="54.0" velocity="6.28"/>
@@ -212,4 +210,5 @@
     <link name="${prefix}wrist_1_link">
       <visual>
+        <origin xyz="0 0 -0.135" rpy="${pi/2} 0 0"/>
         <geometry>
           <mesh filename="package://ur_e_description/meshes/ur10e/visual/wrist1.dae"/>
@@ -220,10 +219,11 @@
       </visual>
       <collision>
+        <origin xyz="0 0 -0.135" rpy="${pi/2} 0 0"/>
         <geometry>
           <mesh filename="package://ur_e_description/meshes/ur10e/collision/wrist1.stl"/>
         </geometry>
       </collision>
-      <xacro:cylinder_inertial radius="0.075" length="0.12" mass="${wrist_1_mass}">
-        <origin xyz="0.0 ${wrist_1_length} 0.0" rpy="0 0 0" />
+      <xacro:cylinder_inertial radius="0.075" length="${-1*__kinematics['wrist_2']['y']}" mass="${wrist_1_mass}">
+        <origin xyz="0.0 0.0 0.0" rpy="0 0 0" />
       </xacro:cylinder_inertial>
     </link>
@@ -231,5 +231,5 @@
       <parent link="${prefix}wrist_1_link" />
       <child link = "${prefix}wrist_2_link" />
-      <origin xyz="0.0 ${wrist_1_length} 0.0" rpy="0.0 0.0 0.0" />
+      <origin xyz="${__kinematics['wrist_2']['x']} ${__kinematics['wrist_2']['y']} ${__kinematics['wrist_2']['z']}" rpy="${__kinematics['wrist_2']['roll']} ${__kinematics['wrist_2']['pitch']} ${__kinematics['wrist_2']['yaw']}" />
       <axis xyz="0 0 1" />
       <xacro:unless value="${joint_limited}">
@@ -249,4 +249,5 @@
     <link name="${prefix}wrist_2_link">
       <visual>
+        <origin xyz="0 0 -0.12" rpy="0 0 0"/>
         <geometry>
           <mesh filename="package://ur_e_description/meshes/ur10e/visual/wrist2.dae"/>
@@ -257,10 +258,11 @@
       </visual>
       <collision>
+        <origin xyz="0 0 -0.12" rpy="0 0 0"/>
         <geometry>
           <mesh filename="package://ur_e_description/meshes/ur10e/collision/wrist2.stl"/>
         </geometry>
       </collision>
-      <xacro:cylinder_inertial radius="0.075" length="0.12" mass="${wrist_2_mass}">
-        <origin xyz="0.0 0.0 ${wrist_2_length}" rpy="0 0 0" />
+      <xacro:cylinder_inertial radius="0.075" length="${__kinematics['wrist_3']['y']}" mass="${wrist_2_mass}">
+        <origin xyz="0.0 0.0 0.0" rpy="0 0 0" />
       </xacro:cylinder_inertial>
     </link>
@@ -268,6 +270,6 @@
       <parent link="${prefix}wrist_2_link" />
       <child link = "${prefix}wrist_3_link" />
-      <origin xyz="0.0 0.0 ${wrist_2_length}" rpy="0.0 0.0 0.0" />
-      <axis xyz="0 1 0" />
+      <origin xyz="${__kinematics['wrist_3']['x']} ${__kinematics['wrist_3']['y']} ${__kinematics['wrist_3']['z']}" rpy="${__kinematics['wrist_3']['roll']} ${__kinematics['wrist_3']['pitch']} ${__kinematics['wrist_3']['yaw']}" />
+      <axis xyz="0 0 1" />
       <xacro:unless value="${joint_limited}">
         <limit lower="${-2.0 * pi}" upper="${2.0 * pi}" effort="54.0" velocity="6.28"/>
@@ -286,4 +288,5 @@
     <link name="${prefix}wrist_3_link">
       <visual>
+        <origin xyz="0 0 -0.1168" rpy="${pi/2} 0 0"/>
         <geometry>
           <mesh filename="package://ur_e_description/meshes/ur10e/visual/wrist3.dae"/>
@@ -294,4 +297,5 @@
       </visual>
       <collision>
+        <origin xyz="0 0 -0.1168" rpy="${pi/2} 0 0"/>
         <geometry>
           <mesh filename="package://ur_e_description/meshes/ur10e/collision/wrist3.stl"/>
@@ -299,5 +303,5 @@
       </collision>
       <xacro:cylinder_inertial radius="0.045" length="0.05" mass="${wrist_3_mass}">
-        <origin xyz="0.0 ${wrist_3_length - 0.05/2} 0.0" rpy="${pi/2} 0 0" />
+        <origin xyz="0.0 0.0 ${-0.05/2}" rpy="0 0 0" />
       </xacro:cylinder_inertial>
     </link>
@@ -305,5 +309,5 @@
       <parent link="${prefix}wrist_3_link" />
       <child link = "${prefix}ee_link" />
-      <origin xyz="0.0 ${wrist_3_length} 0.0" rpy="0.0 0.0 ${pi/2.0}" />
+      <origin xyz="0.0 0.0 0.0" rpy="0.0 ${-pi/2.0} ${pi/2.0}" />
     </joint>
     <link name="${prefix}ee_link">
@@ -324,5 +328,5 @@
                  degrees)
       -->
-      <origin xyz="0 0 0" rpy="0 0 ${-pi}"/>
+      <origin xyz="0 0 0" rpy="0 0 ${-base_correction}"/>
       <parent link="${prefix}base_link"/>
       <child link="${prefix}base"/>
@@ -331,5 +335,5 @@
     <link name="${prefix}tool0"/>
     <joint name="${prefix}wrist_3_link-tool0_fixed_joint" type="fixed">
-      <origin xyz="0 ${wrist_3_length} 0" rpy="${pi/-2.0} 0 0"/>
+      <origin xyz="0 0 0" rpy="0 0 0"/>
       <parent link="${prefix}wrist_3_link"/>
       <child link="${prefix}tool0"/>
